Commit message: Modified description for simpler smaller base. Removed incorrect collision for r200 sensor

File: urdf/morph.xacro (robot description, xacro)
@@ -5,5 +5,5 @@
   <xacro:include filename="$(find morph_description)/urdf/common_properties.xacro" />
   <!-- Import all Gazebo-customization elements, including Gazebo colors -->
-  <xacro:include filename="$(find morph_description)/urdf/morph.gazebo" />
+  <!-- <xacro:include filename="$(find morph_description)/urdf/morph.gazebo" /> -->
   <!-- <xacro:include filename="$(find morph_description)/urdf/kinect.xacro" /> -->
   <xacro:include filename="$(find morph_description)/urdf/r200.xacro" />
@@ -40,22 +40,4 @@
       <geometry>
         <box size="${bar_width} ${top_bar_length} ${t_slot_width}"></box>
-      </geometry>
-    </visual>
-    <visual name="back__vertical_beam_left">
-      <origin xyz="-${back_beam_px} -${t_slot_width} ${(back_vertical_beam_hight*.5)+0.115+(1.5*t_slot_width)}" rpy="0 0 -1.57" />
-      <geometry>
-        <box size="${t_slot_width} ${t_slot_width} ${back_vertical_beam_hight}"></box>
-      </geometry>
-    </visual>
-    <visual name="back__vertical_beam_right">
-      <origin xyz="-${back_beam_px} ${t_slot_width} ${(back_vertical_beam_hight*.5)+0.115+(1.5*t_slot_width)}" rpy="0 0 -1.57" />
-      <geometry>
-        <box size="${t_slot_width} ${t_slot_width} ${back_vertical_beam_hight}"></box>
-      </geometry>
-    </visual>
-    <visual name="back_horizontal_beam">
-      <origin xyz="-${back_beam_px} 0 ${(back_vertical_beam_hight)+0.115+(2*t_slot_width)}" rpy="0 0 -1.57" />
-      <geometry>
-        <box size="${back_horizontal_beam_width} ${t_slot_width} ${t_slot_width}"></box>
       </geometry>
     </visual>
@@ -155,5 +137,5 @@
       </geometry>
     </visual>
-    <collision>R
+    <collision>
       <origin rpy="0 0 0" xyz="0 0 0"/>
       <geometry>

File: urdf/morph_properties.xacro (robot description, xacro)
@@ -2,6 +2,6 @@
 <robot xmlns:xacro="http://www.ros.org/wiki/xacro">
 	<xacro:property name="bottom_bar_length" value="0.128" /> <!-- total distance between two wheels including some space between the bar and the wheel -->
-  <xacro:property name="top_bar_length" value="0.34" />
-	<xacro:property name="top_bar_offset" value="-0.055" />
+  <xacro:property name="top_bar_length" value="0.30" />
+	<xacro:property name="top_bar_offset" value="0.0" />
 	<xacro:property name="bar_width" value="0.06" />
 	<xacro:property name="wheel_radius" value="0.0825" />

File: urdf/r200.xacro (robot description, xacro)
@@ -83,10 +83,4 @@
         </geometry>
       </visual>
-      <collision>
-        <origin xyz="0.0 0.0 0.0" rpy="0 0 0"/>
-        <geometry>
-          <box size="0.130 0.567 0.118"/>
-        </geometry>
-      </collision>-->
       <!-- This inertial field needs doesn't contain reliable data!! -->
      <inertial>

Commit message: Fixed xml namespaces and changed camera position

File: urdf/morph.xacro (robot description, xacro)
@@ -1,4 +1,4 @@
 <?xml version="1.0"?>
-<robot name="morph" xmlns:xacro="http://www.ros.org/wiki/xacro">
+<robot name="morph" xmlns:xacro="http://ros.org/wiki/xacro">
   <xacro:include filename="$(find morph_description)/urdf/morph_properties.xacro" />
   <!-- Import Rviz colors -->
@@ -123,5 +123,5 @@
     <parent link="base_link" />
     <child link="imu_base" />
-    <origin xyz="0.06 -0.02 0.16" rpy="0 0 0" />
+    <origin xyz="-0.06 -0.02 0.16" rpy="0 0 0" />
   </joint>
   <link name="imu_base">

File: urdf/morph_properties.xacro (robot description, xacro)
@@ -1,10 +1,10 @@
 <?xml version="1.0"?>
-<robot xmlns:xacro="http://www.ros.org/wiki/xacro">
-	<xacro:property name="bottom_bar_length" value="0.128" /> <!-- total distance between two wheels including some space between the bar and the wheel -->
+<robot xmlns:xacro="http://ros.org/wiki/xacro">
+	<xacro:property name="bottom_bar_length" value="0.13" /> <!-- total distance between two wheels including some space between the bar and the wheel -->
   <xacro:property name="top_bar_length" value="0.30" />
 	<xacro:property name="top_bar_offset" value="0.0" />
 	<xacro:property name="bar_width" value="0.06" />
-	<xacro:property name="wheel_radius" value="0.0825" />
-	<xacro:property name="wheel_width" value="0.060" /> <!-- total width of the wheel, including wheel surface area (actual tire) and hub portion that stands out-->
+	<xacro:property name="wheel_radius" value="0.085625359" />
+	<xacro:property name="wheel_width" value="0.045" /> <!-- total width of the wheel, including wheel surface area (actual tire) and hub portion that stands out-->
 	<xacro:property name="wheel_mass" value="5.0" />
 	<xacro:property name="caster_radius" value="0.0575" />

File: urdf/r200.xacro (robot description, xacro)
@@ -4,7 +4,7 @@
   <xacro:include filename="$(find turtlebot_description)/urdf/turtlebot_properties.urdf.xacro"/>
   <!-- Mount and camera parameters -->
-  <xacro:property name="pole_px" value="0.08" />
+  <xacro:property name="pole_px" value="0.163" />
   <xacro:property name="pole_py" value="-0.10"/>
-  <xacro:property name="pole_pz" value="${0.08 + t_slot_width + t_slot_width}" />
+  <xacro:property name="pole_pz" value="0.215" />
   <xacro:property name="r200_bracket_end_offset_py" value="0.02" />
   <xacro:property name="r200_bracket_end_offset_pz" value="0" />
