Commit message: Updated morph_properties to match M1-C1 base

File: urdf/morph_properties.xacro (robot description, xacro)
@@ -1,5 +1,5 @@
 <?xml version="1.0"?>
 <robot xmlns:xacro="http://ros.org/wiki/xacro">
-	<xacro:property name="bottom_bar_length" value="0.13" /> <!-- total distance between two wheels including some space between the bar and the wheel -->
+	<xacro:property name="bottom_bar_length" value="0.415" /> <!-- total distance between two wheels including some space between the bar and the wheel -->
   <xacro:property name="top_bar_length" value="0.30" />
 	<xacro:property name="top_bar_offset" value="0.0" />

Commit message: Updated wheel_radius

File: urdf/morph_properties.xacro (robot description, xacro)
@@ -5,5 +5,5 @@
 	<xacro:property name="top_bar_offset" value="0.0" />
 	<xacro:property name="bar_width" value="0.06" />
-	<xacro:property name="wheel_radius" value="0.085625359" />
+	<xacro:property name="wheel_radius" value="0.083238035237061" />
 	<xacro:property name="wheel_width" value="0.045" /> <!-- total width of the wheel, including wheel surface area (actual tire) and hub portion that stands out-->
 	<xacro:property name="wheel_mass" value="5.0" />
